File: bbedison_base/bbedison_base.sch (EAGLE design)
At the start: 4 parts

Commit message: some descriptions was added
Other:
- note added: "Origin of the files: https://github.com/tejonbiker/bbedison Follow US: Federico Ramos @tejonbiker https://tejonbiker.wordpress.com/acerca-de-mi/ Xhabas Jimenez @Sabasacustico http://blog.theinventorhouse.org/"
Changed lines of the file:
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@@
 <sheet>
 <plain>
+<text x="2.54" y="-7.62" size="1.778" layer="94">Origin of the files:
+https://github.com/tejonbiker/bbedison
+Follow US:
+Federico Ramos  @tejonbiker          https://tejonbiker.wordpress.com/acerca-de-mi/
+Xhabas Jimenez  @Sabasacustico   http://blog.theinventorhouse.org/
+</text>
 </plain>
 <instances>
@@
 </schematic>
 </drawing>
+<compatibility>
+<note version="6.3" minversion="6.2.2" severity="warning">
+Since Version 6.2.2 text objects can contain more than one line,
+which will not be processed correctly with this version.
+</note>
+</compatibility>
 </eagle>
